File: project/mouse/mouse.kicad_pcb (KiCad board)
At the start: 2 copper layers, 64 x 72.6 mm, 32 parts, among them J1 Conn_01x06_Male, U1 74LS14, U2 74LS123, U3 74LS123, U4 74LS157, U5 CY7C63231A

Commit message: up
Parts:
- moved R4 16.2 mm to (149.9, 72.8), turned to -90 degrees
- moved D4 12.1 mm to (145.4, 75.0), turned to -90 degrees
- moved C4 12.0 mm to (146.1, 86.4), turned to 180 degrees
Routing:
- net VCC: track 82.2 -> 63.8 mm
- net Net-(U3-Pad13): track 44.0 -> 33.4 mm
- net Net-(C3-Pad1): track 18.9 -> 8.49 mm
- net Net-(C4-Pad1): track 44.0 -> 42.7 mm
- net Net-(U3-Pad5): track 53.3 -> 54.5 mm
- net GND: track 36.1 -> 35.4 mm

Commit message: up
Routing:
- net VCC: track 63.8 -> 163.6 mm, vias 2 -> 3
- net Net-(U3-Pad13): track 33.4 -> 78.3 mm
- net Net-(C3-Pad1): track 8.49 -> 25.4 mm, vias 0 -> 2
- net Net-(C2-Pad1): track 15.1 -> 28.2 mm, vias 1 -> 2
- net Net-(U2-Pad13): track 55.9 -> 68.3 mm
- net Net-(U1-Pad6): track 49.4 -> 43.1 mm
- net Net-(CP2-Pad1): track 93.2 -> 99.1 mm, vias 0 -> 2
- net Net-(U3-Pad5): track 54.5 -> 52.9 mm

Commit message: up
Parts:
- removed the ? at (148.9, 111.0)
- removed G***: LOGO, Library:SimpleKanda_nega
- removed G***: LOGO, Library:SimpleKanda
- moved ? 1.88 mm to (112.1, 45.6)
Routing:
- net VCC: track 163.6 -> 179.6 mm
- net Net-(R5-Pad1): track 23.6 -> 24.6 mm
