File: project/mouse/mouse.kicad_sch (KiCad schematic)
At the start: 24 parts, among them J1 Conn_01x06_Male, U1 74LS14, U2 74LS123, U3 74LS123, U4 74LS157, U5 CY7C63231A

Commit message: up
Parts:
- added U?: PIC18F14K50, symbol AddNew_Library:PIC18F14K50
- added U?: PIC18F14K50-ESO, Package_SO:SOIC-20W_7.5x12.8mm_P1.27mm, symbol MCU_Microchip_PIC18:PIC18F14K50-ESO
